File: Hardware/V1/Credit_card_Midi_piano.kicad_pcb (KiCad board)
At the start: 2 copper layers, 85 x 55 mm, 68 parts, among them J0 0, J1 SJ2-3514A-SMT-TR, J2 0, Q1 BC817-25-QVL, Y301 ABM8G-12.000MHZ-4Y-T3

Commit message: motherboard update
Parts:
- added J3: 0, Resistor_SMD:R_0603_1608Metric, B.Cu at (64.5, 34.1)
- added J4: 0, Resistor_SMD:R_0603_1608Metric, B.Cu at (64.4, 35.8)
- C11, C12, C3, C302, C303, C304, C305, C306, C307, C308, C309, C310, C311, C313, C314, C4, C5, C6, C7, C8, C9, J0, J2, Q1, R1, R10, R11, R12, R13, R14, R2, R3, R305, R313, R314, R4, R5, R6, R7, R8, R9, TP301, TP302, TP303: moved to B.Cu
- moved Q1 61.4 mm to (38.8, 43.6)
- moved C12 59.7 mm to (64.6, 27.4), turned to -90 degrees
- moved C8 55.7 mm to (70.1, 28.2), turned to 90 degrees
- moved BZ1 55.4 mm to (38.2, 42.8), turned to 180 degrees
- moved C11 55.0 mm to (70.7, 30.5), turned to 180 degrees
- moved D1 54.5 mm to (38.3, 37.3), turned to 180 degrees
- moved R13 53.1 mm to (67.1, 28.2), turned to 90 degrees
- moved R12 50.6 mm to (68.8, 28.2), turned to -90 degrees
- moved R14 49.8 mm to (70.1, 32.1), turned to 180 degrees
- moved R7 49.2 mm to (38.5, 46.3), turned to 180 degrees
- moved C7 48.4 mm to (76.1, 30.7), turned to 90 degrees
- moved R9 48.0 mm to (70.5, 24.6), turned to 90 degrees
- moved R8 47.9 mm to (38.7, 40.9), turned to 180 degrees
- moved R11 45.3 mm to (75.6, 22.6), turned to 180 degrees
- moved R304 44.1 mm to (42.0, 22.6), turned to 180 degrees
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Connections:
- net /Controller/3V3 renamed /3V3
- net /Controller/VBUS renamed /VUSB
- BZ1 pad 1: Net-(BZ1-+) -> /VCC_AUDIO
- C9 pad 2: /Audio_out/VCC_Audio -> /VCC_AUDIO
- D1 pad 1: Net-(BZ1-+) -> /VCC_AUDIO
- OP1 pad 8: /Audio_out/VCC_Audio -> /VCC_AUDIO
- Q1 pad 3: Net-(BZ1--) -> Net-(Q1-C)
- R10 pad 1: /Audio_out/VCC_Audio -> /VCC_AUDIO
- R11 pad 1: /Audio_out/VCC_Audio -> /VCC_AUDIO
- R8 pad 1: Net-(BZ1-+) -> Net-(Q1-C)
- R8 pad 2: /Audio_out/VCC_Audio -> Net-(BZ1--)
- uC301 pad 15: /Controller/H4 -> (no net)
- uC301 pad 16: /Controller/H5 -> (no net)
- uC301 pad 17: /Controller/H6 -> (no net)
- uC301 pad 18: /Controller/H7 -> (no net)
- uC301 pad 27: /Controller/cs_sd -> (no net)
- uC301 pad 28: /Controller/cs_lan -> (no net)
Routing:
- net /Controller/QSPI_SS: track 0.00 -> 30.8 mm
- net (no net): track 0.00 -> 25.4 mm, vias 0 -> 2
- net /3V3: track 0.00 -> 23.6 mm, vias 0 -> 9
- net +1V1: track 0.00 -> 21.9 mm, vias 0 -> 3
- net GND: track 0.00 -> 21.7 mm, vias 0 -> 25
- net /Controller/QSPI_SD1: track 0.00 -> 18.4 mm
- net /Controller/QSPI_SD2: track 0.00 -> 14.2 mm
- net /Controller/QSPI_SD3: track 0.00 -> 9.04 mm
- net /Controller/QSPI_SCLK: track 0.00 -> 7.99 mm
- net /VUSB: track 0.00 -> 7.68 mm
- net /Controller/~{USB_BOOT}: track 0.00 -> 7.28 mm
- net Net-(BZ1--): track 0.00 -> 7.17 mm, vias 0 -> 1
- net /Controller/QSPI_SD0: track 0.00 -> 6.97 mm
- net /Controller/USB_D+: track 0.00 -> 5.44 mm
- net /Controller/USB_D-: track 0.00 -> 4.75 mm
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- added copper zone on B.Cu, net /3V3
- added copper zone on F.Cu, net /Audio_out/ADC_Micro
- added copper zone on F.Cu, net /Controller/A2
- added copper zone on F.Cu, net /Controller/GIO21
- added copper zone on F.Cu, net GND
Other:
- outline, holes or cut-outs redrawn
- board text added: "Raster mec: 1mm net: 0.1mm"

Commit message: added keys
Parts:
- removed RN1: CAT10-103J4LF, SamacSys_Parts:CAT10J4LF
- removed TP301, TP302, TP303: TestPoint, TestPoint:TestPoint_Pad_D1.0mm
- removed uC301: SC0914_7_, SamacSys_Parts:QFN40P700X700X90-57N-D
- added H1: Ground_Pen, MountingHole:MountingHole_3.2mm_M3_Pad_Via, F.Cu at (110.8, 41.7)
- added H2: VCC_PEN, MountingHole:MountingHole_3.2mm_M3_Pad_Via, F.Cu at (101.3, 41.8)
- added J5: MEM2085-00-115-00-A, SamacSys_Parts:MEM20850011500A, F.Cu at (86.2, 28.8)
- added JuC1: SC0914_7_, SamacSys_Parts:QFN40P700X700X90-57N-D, F.Cu at (48.9, 39.0)
- R0, R301, R304: moved to B.Cu
- moved R7 41.1 mm to (78.6, 37.4), turned to -90 degrees
- moved Q1 37.6 mm to (75.9, 37.1), turned to 90 degrees
- moved R8 34.7 mm to (73.2, 37.2), turned to -90 degrees
- moved BZ1 23.2 mm to (61.0, 46.9), turned to -90 degrees
- moved D1 19.6 mm to (55.5, 46.8), turned to -90 degrees
- moved C310 10.0 mm to (48.0, 35.6)
- moved C309 9.40 mm to (48.0, 34.3)
- moved R314 9.34 mm to (46.9, 29.2), turned to 0 degrees
- moved R313 9.31 mm to (56.1, 29.3), turned to 180 degrees
- moved C317 6.94 mm to (51.1, 48.4)
- moved R312 6.63 mm to (52.6, 48.0), turned to 90 degrees
- moved R304 6.48 mm to (36.2, 25.4), turned to 0 degrees
- moved R301 5.34 mm to (36.2, 27.1), turned to 180 degrees
- moved C316 4.05 mm to (46.3, 47.5)
- moved J1 2.49 mm to (105.2, 27.0)
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Connections:
- 5sys0 pad 2: (no net) -> Net-(5sys0-A)
- C308 pad 1: (no net) -> Net-(JuC1-ADC_AVDD)
- C317 pad 1: (no net) -> Net-(C317-Pad1)
- R0 pad 1: (no net) -> Net-(5sys0-A)
- R0 pad 2: (no net) -> Net-(JuC1-GPIO23)
- R302 pad 2: (no net) -> Net-(JuC1-USB_DP)
- R303 pad 2: (no net) -> Net-(JuC1-USB_DM)
- R305 pad 2: (no net) -> Net-(JuC1-ADC_AVDD)
- R312 pad 1: (no net) -> Net-(C317-Pad1)
- R313 pad 2: (no net) -> Net-(USB_C301-CC1)
- R314 pad 2: (no net) -> Net-(USB_C301-CC2)
- USB_C301 pad A5: (no net) -> Net-(USB_C301-CC1)
- USB_C301 pad A8: (no net) -> unconnected-(USB_C301-SBU1-PadA8)
- USB_C301 pad B5: (no net) -> Net-(USB_C301-CC2)
- USB_C301 pad B8: (no net) -> unconnected-(USB_C301-SBU2-PadB8)
- Y301 pad 1: (no net) -> Net-(C317-Pad1)
Routing:
- net unconnected-(JuC1-GPIO14-Pad17): track 0.00 -> 85.4 mm, vias 0 -> 2
- net unconnected-(JuC1-GPIO19-Pad30): track 0.00 -> 79.1 mm
- net unconnected-(JuC1-GPIO15-Pad18): track 0.00 -> 65.2 mm, vias 0 -> 2
- net unconnected-(JuC1-GPIO18-Pad29): track 0.00 -> 64.6 mm
- net unconnected-(JuC1-GPIO17-Pad28): track 0.00 -> 60.8 mm
- net unconnected-(JuC1-GPIO13-Pad16): track 0.00 -> 58.2 mm, vias 0 -> 2
- net unconnected-(JuC1-GPIO16-Pad27): track 0.00 -> 58.0 mm
- net unconnected-(JuC1-GPIO12-Pad15): track 0.00 -> 54.1 mm, vias 0 -> 2
- net unconnected-(JuC1-GPIO11-Pad14): track 0.00 -> 50.4 mm, vias 0 -> 2
- net unconnected-(JuC1-GPIO10-Pad13): track 0.00 -> 48.2 mm, vias 0 -> 2
- net unconnected-(JuC1-GPIO9-Pad12): track 0.00 -> 46.6 mm
- net unconnected-(JuC1-GPIO5-Pad7): track 0.00 -> 46.2 mm
- net unconnected-(JuC1-GPIO8-Pad11): track 0.00 -> 43.9 mm
- net unconnected-(JuC1-GPIO7-Pad9): track 0.00 -> 42.4 mm
- net unconnected-(JuC1-GPIO6-Pad8): track 0.00 -> 39.2 mm
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- added copper zone on F.Cu, net (none)
- added copper zone on B.Cu, net GND
- removed copper zone on F.Cu, net /Audio_out/ADC_Micro
- removed copper zone on F.Cu, net /Controller/A2
- removed copper zone on F.Cu, net /Controller/GIO21

Commit message: refined footprint
Parts:
- removed J5: MEM2085-00-115-00-A, SamacSys_Parts:MEM20850011500A
- added C101: 2u2, Capacitor_SMD:C_0805_2012Metric_Pad1.18x1.45mm_HandSolder, B.Cu at (80.8, 22.2)
- added C102: 0.1u, Capacitor_SMD:C_0402_1005Metric_Pad0.74x0.62mm_HandSolder, B.Cu at (86.4, 21.2)
- added J101: MEM2085-00-115-00-A, SamacSys_Parts:MEM20850011500A, F.Cu at (86.4, 27.9)
- added R101: 10k, Resistor_SMD:R_0603_1608Metric_Pad0.98x0.95mm_HandSolder, B.Cu at (89.1, 34.3)
- added R102: 10k, Resistor_SMD:R_0603_1608Metric_Pad0.98x0.95mm_HandSolder, B.Cu at (87.4, 34.3)
- added R103: 10k, Resistor_SMD:R_0603_1608Metric_Pad0.98x0.95mm_HandSolder, B.Cu at (85.7, 34.3)
- added R104: 10k, Resistor_SMD:R_0603_1608Metric_Pad0.98x0.95mm_HandSolder, B.Cu at (84.1, 34.3)
- C9: moved to F.Cu
- moved R7 25.3 mm to (55.4, 47.4), turned to 90 degrees
- moved Q1 20.7 mm to (58.1, 47.7), turned to -90 degrees
- moved R8 16.2 mm to (60.8, 47.6), turned to 90 degrees
- moved J3 8.93 mm to (66.9, 25.5)
- moved J4 8.93 mm to (66.8, 27.2)
- moved C8 8.80 mm to (78.9, 27.9)
- moved R13 6.99 mm to (74.0, 27.6)
- moved C12 6.99 mm to (71.6, 26.8)
- moved R12 6.99 mm to (75.8, 27.6)
- moved C9 6.56 mm to (71.5, 30.2), turned to 180 degrees
- moved R14 5.06 mm to (74.9, 33.6), turned to 0 degrees
- moved C7 5.01 mm to (80.2, 27.9)
- moved C11 4.47 mm to (74.9, 32.0), turned to 0 degrees
- moved R9 4.43 mm to (74.9, 25.0), turned to 180 degrees
- moved J2 2.96 mm to (76.7, 30.4)
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Connections:
- net Net-(C11-Pad2) renamed /Audio_out/opout
- net Net-(OP1A-+) renamed /Audio_out/op+
- net Net-(OP1A--) renamed /Audio_out/op-
Routing:
- net /VCC_AUDIO: track 0.00 -> 58.9 mm, vias 0 -> 2
- net /Audio_out/SLEEVE: track 0.00 -> 29.3 mm, vias 0 -> 1
- net /Audio_out/TIP: track 0.00 -> 26.2 mm, vias 0 -> 1
- net /VUSB: track 6.66 -> 30.6 mm, vias 0 -> 2
- net /Audio_out/RING_1: track 0.00 -> 18.3 mm, vias 0 -> 1
- net GND: track 47.6 -> 65.0 mm, vias 30 -> 39
- net /miso_sd: track 0.00 -> 14.4 mm, vias 0 -> 1
- net /cs_sd: track 0.00 -> 13.9 mm, vias 0 -> 1
- net /mosi_sd: track 0.00 -> 13.3 mm, vias 0 -> 1
- net /sck_sd: track 0.00 -> 13.2 mm, vias 0 -> 1
- net /3V3: track 41.1 -> 51.9 mm, vias 10 -> 14
- net /Audio_out/op+: track 0.00 -> 8.97 mm, vias 0 -> 1
- net /Audio_out/opout: track 0.00 -> 8.27 mm, vias 0 -> 1
- net Net-(BZ1--): track 1.29 -> 9.54 mm, vias 0 -> 1
- net /Audio_out/op-: track 0.00 -> 6.58 mm, vias 0 -> 1
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
Commit message: a
Parts:
- removed C1, C2: 10u, Capacitor_SMD:C_0805_2012Metric_Pad1.18x1.45mm_HandSolder
- removed C101: 2u2, Capacitor_SMD:C_0805_2012Metric_Pad1.18x1.45mm_HandSolder
- removed C102: 0.1u, Capacitor_SMD:C_0402_1005Metric_Pad0.74x0.62mm_HandSolder
- removed J101: MEM2085-00-115-00-A, SamacSys_Parts:MEM20850011500A
- removed J2: 0, Resistor_SMD:R_0603_1608Metric
- removed LRuC1: NCP1117ST33T3G, SamacSys_Parts:SOT230P700X180-4N
- removed R101, R102, R103, R104: 10k, Resistor_SMD:R_0603_1608Metric_Pad0.98x0.95mm_HandSolder
- removed R305: 150, Resistor_SMD:R_0603_1608Metric_Pad0.98x0.95mm_HandSolder
- removed S_BOOT301: 435441019830, SamacSys_Parts:435441019830
- added C10: 47u, Capacitor_SMD:C_1206_3216Metric_Pad1.33x1.80mm_HandSolder, B.Cu at (71.6, 26.8)
- added C13: 2u2, Capacitor_SMD:C_0805_2012Metric_Pad1.18x1.45mm_HandSolder, B.Cu at (80.8, 22.2)
- added C14: 2u2, Capacitor_SMD:C_0805_2012Metric_Pad1.18x1.45mm_HandSolder, B.Cu at (66.2, 30.8)
- added C15: 2u2, Capacitor_SMD:C_0805_2012Metric_Pad1.18x1.45mm_HandSolder, B.Cu at (61.0, 31.6)
- added IC1: MIC5528-3.3YMT-TR, SamacSys_Parts:SON40P120X120X60-7N-D, B.Cu at (63.5, 31.0)
- added J5: MEM2085-00-115-00-A, SamacSys_Parts:MEM20850011500A, F.Cu at (88.0, 25.2)
- added J_Mic1: 0, Resistor_SMD:R_0603_1608Metric, B.Cu at (76.8, 30.1)
- added R15: 10k, Resistor_SMD:R_0603_1608Metric_Pad0.98x0.95mm_HandSolder, B.Cu at (81.0, 37.6)
- added R16: 10k, Resistor_SMD:R_0603_1608Metric_Pad0.98x0.95mm_HandSolder, B.Cu at (82.8, 37.6)
- added R17: 10k, Resistor_SMD:R_0603_1608Metric_Pad0.98x0.95mm_HandSolder, B.Cu at (79.2, 37.6)
- added R18: 10k, Resistor_SMD:R_0603_1608Metric_Pad0.98x0.95mm_HandSolder, B.Cu at (77.4, 37.6)
- added S1: TS20-42-25-WT-160-SMT-TR, SamacSys_Parts:TS204225WT160SMTTR, F.Cu at (38.4, 24.8)
- added S2: TS20-42-25-WT-160-SMT-TR, SamacSys_Parts:TS204225WT160SMTTR, F.Cu at (79.0, 43.6)
- added S3: TS20-42-25-WT-160-SMT-TR, SamacSys_Parts:TS204225WT160SMTTR, F.Cu at (70.8, 43.6)
- C11, C7, C8: footprint Capacitor_SMD:C_0402_1005Metric -> Capacitor_SMD:C_0805_2012Metric_Pad1.18x1.45mm_HandSolder
- C12: value 47u -> 0.1u; footprint Capacitor_SMD:C_1206_3216Metric_Pad1.33x1.80mm_HandSolder -> Capacitor_SMD:C_0402_1005Metric_Pad0.74x0.62mm_HandSolder
- moved C12 15.8 mm to (86.4, 21.2), turned to 0 degrees
- moved 5sys0 3.95 mm to (62.6, 39.4), turned to 180 degrees
- moved C313 2.89 mm to (48.0, 41.5), turned to 180 degrees
- moved R4 2.62 mm to (85.1, 31.3), turned to 180 degrees
- moved R0 2.50 mm to (60.6, 38.8)
- moved C7 0.89 mm to (81.0, 27.5)
- moved C8 0.40 mm to (78.9, 27.5)
- moved R14 0.25 mm to (74.9, 33.9)
- moved R1 0.20 mm to (83.0, 24.7)
Connections:
- C12 pad 1: GND -> /3V3
- C12 pad 2: Net-(C12-Pad2) -> GND
- C308 pad 1: Net-(JuC1-ADC_AVDD) -> /3V3
- JuC1 pad 31: unconnected-(JuC1-GPIO20-Pad31) -> Net-(JuC1-GPIO20)
- JuC1 pad 32: unconnected-(JuC1-GPIO21-Pad32) -> Net-(JuC1-GPIO21)
- JuC1 pad 34: unconnected-(JuC1-GPIO22-Pad34) -> Net-(JuC1-GPIO22)
- JuC1 pad 35: Net-(JuC1-GPIO23) -> /Audio_out/Audio_right
- JuC1 pad 36: unconnected-(JuC1-GPIO24-Pad36) -> /Controller/SPI_MOSI
- JuC1 pad 37: unconnected-(JuC1-GPIO25-Pad37) -> /Controller/SPI_CS
- JuC1 pad 38: unconnected-(JuC1-GPIO26/ADC0-Pad38) -> /Controller/SPI_SCK
- JuC1 pad 39: /Controller/A1 -> /Controller/SPI_MISO
- JuC1 pad 40: /Controller/A2 -> /Audio_out/Audio_left
- JuC1 pad 41: /Controller/A3 -> /Audio_out/ADC_Micro
- JuC1 pad 43: Net-(JuC1-ADC_AVDD) -> /3V3
- OP1 pad 5: (no net) -> GND
- OP1 pad 6: (no net) -> GND
- OP1 pad 7: (no net) -> unconnected-(OP1-Pad7)
- R0 pad 2: Net-(JuC1-GPIO23) -> Net-(JuC1-GPIO22)
- R13 pad 1: Net-(C12-Pad2) -> Net-(C10-Pad2)
Routing:
- net /Controller/SPI_CS: track 0.00 -> 46.9 mm, vias 0 -> 1
- net /Controller/SPI_MOSI: track 0.00 -> 44.2 mm, vias 0 -> 1
- net /Controller/SPI_SCK: track 0.00 -> 41.7 mm, vias 0 -> 1
- net /Audio_out/Audio_right: track 0.00 -> 40.3 mm, vias 0 -> 1
- net /Controller/SPI_MISO: track 0.00 -> 39.0 mm, vias 0 -> 1
- net /Audio_out/Audio_left: track 0.00 -> 38.6 mm, vias 0 -> 1
- net Net-(JuC1-GPIO21): track 0.00 -> 30.5 mm
- net /Audio_out/ADC_Micro: track 1.78 -> 25.2 mm, vias 0 -> 1
- net Net-(JuC1-GPIO20): track 0.00 -> 21.2 mm
- net /miso_sd: track 14.4 -> 0.00 mm, vias 1 -> 0
- net /cs_sd: track 13.9 -> 0.00 mm, vias 1 -> 0
- net /mosi_sd: track 13.3 -> 0.00 mm, vias 1 -> 0
- net /sck_sd: track 13.2 -> 0.00 mm, vias 1 -> 0
- net GND: track 65.0 -> 77.5 mm, vias 39 -> 44
- net unconnected-(JuC1-GPIO25-Pad37): track 9.56 -> 0.00 mm
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Other:
- board text added: "How do you know when a jazz singer is at your door? They can't find the key and don't know when to come in."
- board text added: "How many jazz musicians does it take to change a lightbulb? Five: One to change the bulb and the other four to talk about how Miles Davis would have done it."
- board text added: "J_MICAMP"
- board text added: "J_MONO"
- board text added: "STYRO LOLA"
- board text added: "Stylus 1"
- board text added: "Stylus 2"
- board text added: "What did the jazz saxophonist say when he saw the set list? {dblquote}These are all just notes, not numbers!{dblquote}"
- board text added: "What do y call a jazz musician without partner? homeless"
- board text added: "What is the difference between a jazz singer and a pizza? a pizza can feed a family of four"
- board text added: "key+ key- pause resumne"
- board text added: "or a mp3 player or a synth to go or a drum mashine"
- board text added: "reset boot"

Commit message: asd
Parts:
- removed C301, C304, C307, C308: 2u2, Capacitor_SMD:C_0805_2012Metric_Pad1.18x1.45mm_HandSolder
- removed H1: Ground_Pen, MountingHole:MountingHole_3.2mm_M3_Pad_Via
- removed H2: VCC_PEN, MountingHole:MountingHole_3.2mm_M3_Pad_Via
- removed J0, J3, J4, J_Mic1: 0, Resistor_SMD:R_0603_1608Metric
- removed OP1: TLV9002QDRQ1, SamacSys_Parts:SOIC127P600X175-8N
- removed R10: 5.9k, Resistor_SMD:R_0603_1608Metric_Pad0.98x0.95mm_HandSolder
- removed R11, R9: 200k, Resistor_SMD:R_0603_1608Metric_Pad0.98x0.95mm_HandSolder
- removed R12, R14: 10k, Resistor_SMD:R_0603_1608Metric_Pad0.98x0.95mm_HandSolder
- removed R13: 787, Resistor_SMD:R_0603_1608Metric_Pad0.98x0.95mm_HandSolder
- removed R6: 1.8k, Resistor_SMD:R_0603_1608Metric
- added C1: 2u2, SamacSys_Parts:CAPC1608X90N, B.Cu at (51.0, 32.0)
- added C16: 2u2, SamacSys_Parts:CAPC1608X90N, B.Cu at (75.8, 25.0)
- added C17: 10u, SamacSys_Parts:CAPC1608X50N, B.Cu at (59.7, 25.4)
- added C18: 0.1uF, Capacitor_SMD:C_0402_1005Metric_Pad0.74x0.62mm_HandSolder, B.Cu at (78.0, 23.4)
- added C19: 10u, SamacSys_Parts:CAPC1608X50N, B.Cu at (75.6, 28.8)
- added C2: 2u2, SamacSys_Parts:CAPC1608X90N, B.Cu at (53.5, 32.7)
- added C20: 0.1uF, Capacitor_SMD:C_0402_1005Metric_Pad0.74x0.62mm_HandSolder, B.Cu at (74.4, 25.1)
- added C21: 2u2, SamacSys_Parts:CAPC1608X90N, B.Cu at (84.9, 23.5)
- added C22: 10u, SamacSys_Parts:CAPC1608X50N, B.Cu at (71.0, 27.8)
- added C24: 10u, SamacSys_Parts:CAPC1608X50N, B.Cu at (59.7, 22.7)
- added IC2: MCP73831T-2ACI_OT, SamacSys_Parts:SOT95P270X145-5N, B.Cu at (62.5, 23.3)
- added IC3: PCM5101APWR, Package_SO:TSSOP-20_4.4x6.5mm_P0.65mm, F.Cu at (74.8, 26.7)
- added IC4: MIC5528-3.3YMT-TR, SamacSys_Parts:SON40P120X120X60-7N-D, B.Cu at (66.8, 31.6)
- added PEN_CON1: 502352-0200, SamacSys_Parts:5023520200, F.Cu at (103.5, 41.4)
- C10, C6: value 47u -> 2u2; footprint Capacitor_SMD:C_1206_3216Metric_Pad1.33x1.80mm_HandSolder -> SamacSys_Parts:CAPC1608X90N
- C11: value 3.3u -> 2u2; footprint Capacitor_SMD:C_0805_2012Metric_Pad1.18x1.45mm_HandSolder -> SamacSys_Parts:CAPC1608X90N
- C13, C14, C15: footprint Capacitor_SMD:C_0805_2012Metric_Pad1.18x1.45mm_HandSolder -> SamacSys_Parts:CAPC1608X90N
- C3: value 47u -> 0.1uF; footprint Capacitor_SMD:C_1206_3216Metric_Pad1.33x1.80mm_HandSolder -> Capacitor_SMD:C_0402_1005Metric_Pad0.74x0.62mm_HandSolder
- C4: value 0.1u -> 10u; footprint Capacitor_SMD:C_0402_1005Metric -> SamacSys_Parts:CAPC1608X50N
- C5: value 0.1u -> 0.1uF; footprint Capacitor_SMD:C_0402_1005Metric -> Capacitor_SMD:C_0402_1005Metric_Pad0.74x0.62mm_HandSolder
- C7: value 330n -> 2u2; footprint Capacitor_SMD:C_0805_2012Metric_Pad1.18x1.45mm_HandSolder -> SamacSys_Parts:CAPC1608X90N
- C8: value 120p -> 2u2; footprint Capacitor_SMD:C_0805_2012Metric_Pad1.18x1.45mm_HandSolder -> SamacSys_Parts:CAPC1608X90N
- C9: value 0.1uF -> 2u2; footprint Capacitor_SMD:C_0402_1005Metric_Pad0.74x0.62mm_HandSolder -> SamacSys_Parts:CAPC1608X90N; moved to B.Cu
- J1: value SJ2-3514A-SMT-TR -> SJ2-35853B-SMT-TR; footprint SamacSys_Parts:SJ23514ASMTTR -> SamacSys_Parts:SJ235853BSMTTR
- R1: value 220 -> 470; footprint Resistor_SMD:R_0603_1608Metric -> Resistor_SMD:R_0603_1608Metric_Pad0.98x0.95mm_HandSolder
- R2: value 100 -> 470; footprint Resistor_SMD:R_0603_1608Metric -> Resistor_SMD:R_0603_1608Metric_Pad0.98x0.95mm_HandSolder
- R3: value 1.8k -> 100k
- R4: value 220 -> 2kOhm; footprint Resistor_SMD:R_0603_1608Metric -> Resistor_SMD:R_0603_1608Metric_Pad0.98x0.95mm_HandSolder
- R5: value 100 -> 100k; footprint Resistor_SMD:R_0603_1608Metric -> Resistor_SMD:R_0603_1608Metric_Pad0.98x0.95mm_HandSolder
- R7, R8: value 220 -> ToDo
- moved R3 37.4 mm to (61.1, 38.5), turned to 0 degrees
- moved 5sys0 24.7 mm to (43.3, 24.0), turned to -90 degrees
- moved C15 24.5 mm to (84.9, 26.6), turned to -90 degrees
- moved C14 23.5 mm to (43.2, 25.9)
- moved R5 23.4 mm to (62.5, 26.5), turned to 180 degrees
- moved R0 23.1 mm to (41.6, 25.6), turned to -90 degrees
- moved C3 22.1 mm to (69.6, 27.8), turned to -90 degrees
- moved R4 21.4 mm to (65.2, 23.4), turned to 90 degrees
- moved C9 16.7 mm to (55.0, 32.7), turned to 90 degrees
- moved C7 14.6 mm to (66.5, 29.4), turned to 180 degrees
- moved C8 13.8 mm to (66.6, 33.8), turned to 180 degrees
- moved C11 13.4 mm to (61.8, 29.4), turned to 180 degrees
- moved C5 13.2 mm to (74.4, 28.8), turned to -90 degrees
- moved C10 11.9 mm to (61.9, 33.6), turned to 180 degrees
- moved C13 11.4 mm to (89.4, 29.7), turned to -90 degrees
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Connections:
- BZ1 pad 1: /VCC_AUDIO -> /V_SYS
- C10 pad 1: GND -> /3V3
- C10 pad 2: Net-(C10-Pad2) -> GND
- C11 pad 1: /Audio_out/ADC_Micro -> /V_SYS
- C11 pad 2: /Audio_out/opout -> GND
- C13 pad 1: GND -> /3V3
- C13 pad 2: /3V3 -> GND
- C14 pad 1: GND -> /3V3
- C14 pad 2: /3V3 -> GND
- C15 pad 1: GND -> /Audio_out/TIP
- C15 pad 2: /VUSB -> GND
- C3 pad 1: Net-(C3-Pad1) -> GND
- C3 pad 2: /Audio_out/TIP -> /3V3
- C4 pad 1: Net-(C3-Pad1) -> /Audio_out/3V3_A
- C5 pad 1: Net-(C5-Pad1) -> GND
- C5 pad 2: GND -> /Audio_out/3V3_A
- C6 pad 1: Net-(C5-Pad1) -> Net-(IC3-CAPP)
- C6 pad 2: /Audio_out/RING_1 -> Net-(IC3-CAPM)
- C7 pad 1: /Audio_out/SLEEVE -> /V_SYS
- C7 pad 2: /Audio_out/op+ -> GND
- C8 pad 1: /Audio_out/opout -> /Audio_out/3V3_A
- C8 pad 2: /Audio_out/op- -> GND
- C9 pad 1: GND -> /3V3
- C9 pad 2: /VCC_AUDIO -> GND
- D1 pad 1: /VCC_AUDIO -> /V_SYS
- IC1 pad 4: /VUSB -> /V_SYS
- IC1 pad 6: /VUSB -> /V_SYS
- J1 pad 1: /Audio_out/SLEEVE -> GND
- J1 pad 3: /Audio_out/RING_1 -> /Audio_out/RING
- JuC1 pad 18: unconnected-(JuC1-GPIO15-Pad18) -> /Controller/GPIO15
- JuC1 pad 2: /Controller/GPIO0 -> unconnected-(JuC1-GPIO0-Pad2)
- JuC1 pad 3: /Controller/GPIO1 -> unconnected-(JuC1-GPIO1-Pad3)
- JuC1 pad 34: Net-(JuC1-GPIO22) -> /Audio_out/Buzzer
- JuC1 pad 35: /Audio_out/Audio_right -> /Audio_out/Audio_0
- JuC1 pad 40: /Audio_out/Audio_left -> /Audio_out/Audio_1
- JuC1 pad 41: /Audio_out/ADC_Micro -> /Audio_out/Audio_2
- R0 pad 2: Net-(JuC1-GPIO22) -> /3V3
- R1 pad 1: /Audio_out/Audio_left -> Net-(IC3-OUTL)
- R1 pad 2: Net-(C3-Pad1) -> /Audio_out/TIP
- R2 pad 1: GND -> Net-(IC3-OUTR)
- R2 pad 2: Net-(C3-Pad1) -> /Audio_out/RING
- R3 pad 1: GND -> /Audio_out/Buzzer
- R3 pad 2: /Audio_out/TIP -> /Audio_out/Headphone_connected
- R4 pad 1: /Audio_out/Audio_right -> GND
- R4 pad 2: Net-(C5-Pad1) -> Net-(IC2-PROG)
- R5 pad 1: GND -> Net-(IC2-STAT)
- R5 pad 2: Net-(C5-Pad1) -> /Controller/GPIO15
- USB_C301 pad A4: /VUSB -> /Controller/VUSB
- USB_C301 pad A9: /VUSB -> /Controller/VUSB
Routing:
- net /Controller/GPIO15: track 0.00 -> 93.1 mm, vias 0 -> 4
- net unconnected-(JuC1-GPIO15-Pad18): track 65.2 -> 0.00 mm, vias 2 -> 0
- net /V_SYS: track 0.00 -> 56.2 mm, vias 0 -> 3
- net /VCC_AUDIO: track 53.1 -> 0.00 mm, vias 3 -> 0
- net /Audio_out/Headphone_connected: track 0.00 -> 51.8 mm, vias 0 -> 1
- net /Audio_out/Audio_right: track 40.3 -> 0.00 mm, vias 1 -> 0
- net /Audio_out/Audio_left: track 38.6 -> 0.00 mm, vias 1 -> 0
- net /VUSB: track 34.7 -> 0.00 mm, vias 1 -> 0
- net /Audio_out/3V3_A: track 0.00 -> 33.4 mm, vias 0 -> 2
- net unconnected-(JuC1-GPIO0-Pad2): track 0.00 -> 31.0 mm
- net /Controller/GPIO0: track 31.0 -> 0.00 mm
- net /Audio_out/Audio_0: track 0.00 -> 30.9 mm, vias 0 -> 2
- net /Audio_out/SLEEVE: track 28.6 -> 0.00 mm, vias 1 -> 0
- net /Audio_out/Audio_2: track 0.00 -> 28.3 mm
- net /Audio_out/Audio_1: track 0.00 -> 28.2 mm
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- added copper zone on B.Cu, net /V_SYS
Other:
- board text added: "0"
- board text added: "1"
- board text added: "AUX"
- board text added: "Audio IC"
- board text added: "Buzzer"
- board text added: "Flash"
- board text added: "Stylus"
- board text added: "USB-C"
- board text removed: "J_MICAMP"
- board text removed: "J_MONO"
- board text removed: "Stylus 1"
- board text removed: "Stylus 2"

Commit message: oi
Routing:
- net GND: track 87.0 -> 89.9 mm, vias 53 -> 51
- net /Audio_out/Headphone_connected: track 51.8 -> 52.8 mm
