File: Hardware/V1/Controller.kicad_sch (KiCad schematic)
At the start: 35 parts, among them IC1 MIC5528-3.3YMT-TR, Y301 ABM8G-12.000MHZ-4Y-T3

Commit message: asd
Parts:
- removed C14, C15, C301, C304, C307, C308: 2u2, Capacitor_SMD:C_0805_2012Metric_Pad1.18x1.45mm_HandSolder, symbol SymbolsBalloonv4:C
- added C1, C10, C11, C14, C2, C9: 2u2, SamacSys_Parts:CAPC1608X90N, symbol Device:C_Small
- added C17, C24: 10u, SamacSys_Parts:CAPC1608X50N, symbol Device:C_Small
- added IC2: MCP73831T-2ACI_OT, SamacSys_Parts:SOT95P270X145-5N, symbol SamacSys_Parts:MCP73831T-2ACI_OT
- added R4: 2kOhm, Resistor_SMD:R_0603_1608Metric_Pad0.98x0.95mm_HandSolder, symbol Device:R_Small
- added R5: 100k, Resistor_SMD:R_0603_1608Metric_Pad0.98x0.95mm_HandSolder, symbol Device:R_Small
- IC1: footprint SON40P120X120X60-7N-D -> SamacSys_Parts:SON40P120X120X60-7N-D
- S1, S2, S3: footprint TS204225WT160SMTTR -> SamacSys_Parts:TS204225WT160SMTTR
Connections:
- net +1V1: now also C1.1
- net 3V3: now also R0.2, C10.1, C14.1, C2.1, C9.1
- net GND: now also C1.2, C10.2, C11.2, C14.2, C17.2, C2.2, C24.2, C9.2, IC2.2 (VSS), R4.1
- net GPIO22: now reaches JuC1.34 (GPIO22)
- net GPIO22: no longer R0.2
- net GPIO15: now reaches JuC1.18 (GPIO15)
- net GPIO15: now also R5.2
- net A1 renamed GPIO23
- net A2 renamed GPIO28
- net A3 renamed GPIO29
- net GPIO0: no longer names the net of JuC1.2 (GPIO0)
- net GPIO1: no longer names the net of JuC1.3 (GPIO1)
- net VBUS renamed VSYS
- net VSYS: now also C11.1, C17.1, IC2.3 (VBAT); no longer USB_C301.A4 (VBUS_1), USB_C301.A9 (VBUS_2)
- new net: IC2.5 (PROG), R4.2
- new net: IC2.1 (STAT), R5.1
- new net VUSB: C24.1, IC2.4 (VDD), USB_C301.A4 (VBUS_1), USB_C301.A9 (VBUS_2)
- no-connect marks 4 -> 23
Other:
- moved on the sheet: 5sys0, IC1, R0

Commit message: changed to make boom better
Parts:
- C302: value 0.1uF -> 0.1u
Changed lines of the file:
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@@
 			)
 		)
-		(property "Value" "0.1uF"
+		(property "Value" "0.1u"
 			(at 73.279 34.163 0)
 			(effects
